File: Current Sensor.kicad_sch (KiCad schematic)
At the start: 4 parts, among them U1 CC6920BSO-5A

Commit message: Working on the layout
Parts:
- renumbered C5 to C7, C4 to C8, R4 to R8, U1 to U4
Other:
- moved on the sheet: C7, C8, R8, U4
