File: Current_Probe_CC6920B.kicad_sch (KiCad schematic)
At the start: 22 parts, among them J1 USB_C_Receptacle_USB2.0, J2 I_IN, J4 EDGE MOUNT SMA, SW1 SLIDE_SPDT, SW2 SLIDE_SPDT, U1 CC6920BSO-5A, U2 TPD4E1U06DCKR, U3 HT7533-1

Commit message: Schematic mostly done?
Parts:
- removed C4: 100nF, Capacitor_SMD:C_0603_1608Metric, symbol Device:C
- removed C5: 220pF, Capacitor_SMD:C_0603_1608Metric, symbol Device:C
- removed R4: 47R, Resistor_SMD:R_0603_1608Metric, symbol Device:R
- removed SW2: SLIDE_SPDT, Button_Switch_SMD:SW_SPDT_PCM12, symbol Switch:SW_SPDT
- removed U1: CC6920BSO-5A, Package_SO:SOIC-8_3.9x4.9mm_P1.27mm, symbol Current_Probe_CC6920B:CC6920BSO-5A
- added C8: 100nF, Capacitor_SMD:C_0603_1608Metric, symbol Device:C
- added J3: Conn_01x05_Pin, Connector_PinHeader_2.54mm:PinHeader_1x05_P2.54mm_Vertical, symbol Connector:Conn_01x05_Pin
- added R8: 330R, Resistor_SMD:R_0603_1608Metric, symbol Device:R
- added SW3: FILT_EN, Button_Switch_SMD:SW_SPDT_PCM12, symbol Switch:SW_SPDT
- J1: symbol Connector:USB_C_Receptacle_USB2.0 -> Connector:USB_C_Receptacle_USB2.0_16P
- SW1: value SLIDE_SPDT -> GAIN_SEL
- U2: symbol CANchovy_PCB:TPD4E1U06DCKR -> Current_Probe_CC6920B:TPD4E1U06DCKR
Connections:
- net +5V: now also J3.5 (Pin_5)
- net GND: now also C8.2, J3.1 (Pin_1)
- net V_AMPLIFIED: now reaches SW1.1 (A)
- net V_AMPLIFIED: now also J3.4 (Pin_4)
- net at SW1.2 (B): now also J4.1 (In)
- net OUT_FILT: now reaches SW1.3 (C)
- net OUT_FILT: now also J3.3 (Pin_3), R8.2, SW3.2 (B)
- net GND_VIRT: now reaches J4.2 (Ext)
- net GND_VIRT: now also J3.2 (Pin_2)
- net Current Sensor/IP+: now reaches J2.2 (Pin_2)
- net Current Sensor/IP-: now reaches J2.1 (Pin_1)
- new net: C8.1, SW3.1 (A)
- new net Current Sensor/OUT: R8.1
- no-connect marks 6 -> 7
Other:
- added sheet Current Sensor (Current Sensor.kicad_sch)
- note added: "-3dB @ ~4.8kHz"
- note added: "3.3V rail indication"
- note added: "Current sensor"
- note added: "Current signal path"
- note added: "Oscilloscope output"
- note added: "Pin header outputs"
- note added: "Power Input"
- note removed: "-3dB ~400kHz"
- moved on the sheet: C1, C2, C3, D1, FB1, J1, J4, R1, R2, R3, R5, SW1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

Commit message: Working on the layout
Parts:
- removed J3: Conn_01x05_Pin, Connector_PinHeader_2.54mm:PinHeader_1x05_P2.54mm_Vertical, symbol Connector:Conn_01x05_Pin
- added TP2, TP3, TP5, TP6, TP7: TestPoint, TestPoint:TestPoint_THTPad_1.0x1.0mm_Drill0.5mm, symbol Connector:TestPoint
- J2: footprint (none) -> TerminalBlock_Phoenix:TerminalBlock_Phoenix_MKDS-1,5-2_1x02_P5.00mm_Horizontal; LCSC Part # (none) -> C8269; Manufacturer (none) -> Ningbo Kangnex Elec; Manufacturer Part # (none) -> WJ128V-5.0-2P
- renumbered C8 to C2, C2 to C3, C3 to C4, J4 to J3, R8 to R4, SW3 to SW1, SW1 to SW2, TP2 to TP4, U2 to U1, U3 to U2
Connections:
- net Current Sensor/IP+: now also J2.1 (Pin_1); no longer J2.2 (Pin_2)
- net Current Sensor/IP-: now also J2.2 (Pin_2); no longer J2.1 (Pin_1)
- net Current Sensor/OUT: now also TP3.1
- net GND: now also TP2.1
- net OUT_FILT: now also TP5.1
- net V_AMPLIFIED: now also TP6.1
- net at J3.1 (In), SW2.2 (B): now also TP7.1
Other:
- note removed: "Pin header outputs"
- moved on the sheet: J2
