File: Amplifier.kicad_sch (KiCad schematic)
At the start: 5 parts, among them U4 COS721

Commit message: Working on the layout
Parts:
- renumbered C6 to C5, C7 to C6, R7 to R6, R6 to R7, U4 to U3
Changed lines of the file:
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@@
 		(on_board yes)
 		(dnp no)
-		(property "Reference" "U4"
+		(property "Reference" "U3"
 			(at 149.86 81.28 0)
 			(effects
@@
 			(project ""
 				(path "/a088a2fb-dae0-46a5-a56c-5b567ab29624/3883a9c1-b4d4-446e-8a12-1b5b82cac23f"
-					(reference "U4")
+					(reference "U3")
 					(unit 1)
 				)
@@
 		(on_board yes)
 		(dnp no)
-		(property "Reference" "R6"
+		(property "Reference" "R7"
 			(at 146.05 113.03 90)
 			(effects
@@
 			(project "Current_Probe_CC6920B"
 				(path "/a088a2fb-dae0-46a5-a56c-5b567ab29624/3883a9c1-b4d4-446e-8a12-1b5b82cac23f"
-					(reference "R6")
+					(reference "R7")
 					(unit 1)
 				)
@@
 		(on_board yes)
 		(dnp yes)
-		(property "Reference" "C7"
+		(property "Reference" "C6"
 			(at 146.05 124.46 90)
 			(effects
@@
 			(project ""
 				(path "/a088a2fb-dae0-46a5-a56c-5b567ab29624/3883a9c1-b4d4-446e-8a12-1b5b82cac23f"
-					(reference "C7")
+					(reference "C6")
 					(unit 1)
 				)
@@
 		(dnp no)
 		(fields_autoplaced yes)
-		(property "Reference" "R7"
+		(property "Reference" "R6"
 			(at 137.16 126.9999 0)
 			(effects
@@
 			(project "Current_Probe_CC6920B"
 				(path "/a088a2fb-dae0-46a5-a56c-5b567ab29624/3883a9c1-b4d4-446e-8a12-1b5b82cac23f"
-					(reference "R7")
+					(reference "R6")
 					(unit 1)
 				)
@@
 		(dnp no)
 		(fields_autoplaced yes)
-		(property "Reference" "C6"
+		(property "Reference" "C5"
 			(at 120.65 106.6799 0)
 			(effects
@@
 			(project "Current_Probe_CC6920B"
 				(path "/a088a2fb-dae0-46a5-a56c-5b567ab29624/3883a9c1-b4d4-446e-8a12-1b5b82cac23f"
-					(reference "C6")
+					(reference "C5")
 					(unit 1)
 				)

Commit message: Rev A sent for manufacture.
Changed lines of the file:
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@@
+		)
+	)
+	(text_box "40A range = 50mV/A\n2x gain = 100mV/A (in 10x probe mode good option for scope)\nRes ratio = 1:1\n\n20A range = 100mV/A\nAlready suitable for scope in 10x mode\n"
+		(exclude_from_sim no)
+		(at 20.32 44.45 0)
+		(size 52.07 16.51)
+		(stroke
+			(width 0)
+			(type default)
+		)
+		(fill
+			(type none)
+		)
+		(effects
+			(font
+				(size 1.27 1.27)
+			)
+			(justify left top)
 		)
 	)
