File: Current_Probe_CC6920B.kicad_pcb (KiCad board)
At the start: 2 copper layers, 28 parts, among them J1 USB_C_Receptacle_USB2.0, J4 EDGE MOUNT SMA, SW1 GAIN_SEL, SW3 FILT_EN, U1 CC6920BSO-5A, U2 TPD4E1U06DCKR, U3 HT7533-1, U4 COS721

Commit message: Working on the layout
Parts:
- removed J4: EDGE MOUNT SMA, Connector_Coaxial:SMA_Samtec_SMA-J-P-H-ST-EM1_EdgeMount
- removed SW3: FILT_EN, Button_Switch_SMD:SW_SPDT_PCM12
- added J2: I_IN, TerminalBlock_Phoenix:TerminalBlock_Phoenix_MKDS-1,5-2_1x02_P5.00mm_Horizontal, F.Cu at (133.7, 90.0)
- added J3: EDGE MOUNT SMA, Connector_Coaxial:SMA_Samtec_SMA-J-P-H-ST-EM1_EdgeMount, F.Cu at (102.1, 95.7)
- added SW2: GAIN_SEL, Button_Switch_SMD:SW_SPDT_PCM12, F.Cu at (109.5, 98.0)
- added TP3: TestPoint, TestPoint:TestPoint_THTPad_1.0x1.0mm_Drill0.5mm, F.Cu at (117.8, 91.4)
- added TP4: TestPoint, TestPoint:TestPoint_THTPad_1.0x1.0mm_Drill0.5mm, F.Cu at (125.5, 79.3)
- added TP5: TestPoint, TestPoint:TestPoint_THTPad_1.0x1.0mm_Drill0.5mm, F.Cu at (112.5, 94.4)
- added TP6: TestPoint, TestPoint:TestPoint_THTPad_1.0x1.0mm_Drill0.5mm, F.Cu at (106.5, 94.4)
- added TP7: TestPoint, TestPoint:TestPoint_THTPad_1.0x1.0mm_Drill0.5mm, F.Cu at (109.5, 94.4)
- C2: value 1uF -> 100nF; footprint Capacitor_SMD:C_0805_2012Metric -> Capacitor_SMD:C_0603_1608Metric
- C3: value 10uF -> 1uF; footprint Capacitor_SMD:C_0603_1608Metric -> Capacitor_SMD:C_0805_2012Metric
- C4: value 220pF -> 10uF
- C6: value 100nF -> C
- C7: value C -> 100nF
- C8: value 100nF -> 220pF
- R4: value 47R -> 330R
- R6: value 12k 0.1% -> 4.3k 0.1%
- R7: value 4.3k 0.1% -> 12k 0.1%
- R8: value 330R -> 47R
- SW1: value GAIN_SEL -> FILT_EN
- U1: value CC6920BSO-5A -> TPD4E1U06DCKR; footprint Package_SO:SOIC-8_3.9x4.9mm_P1.27mm -> Package_TO_SOT_SMD:SOT-363_SC-70-6
- U2: value TPD4E1U06DCKR -> HT7533-1; footprint Package_TO_SOT_SMD:SOT-363_SC-70-6 -> Package_TO_SOT_SMD:SOT-89-3
- U3: value HT7533-1 -> COS721; footprint Package_TO_SOT_SMD:SOT-89-3 -> Package_TO_SOT_SMD:SOT-23-5
- U4: value COS721 -> CC6920BSO-5A; footprint Package_TO_SOT_SMD:SOT-23-5 -> Package_SO:SOIC-8_3.9x4.9mm_P1.27mm
- moved R8 103.7 mm to (117.8, 89.5)
- moved C3 101.9 mm to (121.5, 79.3), turned to -90 degrees
- moved C8 100.5 mm to (117.8, 88.0)
- moved FB1 98.2 mm to (122.0, 76.8)
- moved C2 92.0 mm to (117.2, 94.6), turned to 180 degrees
- moved U3 91.4 mm to (108.3, 89.8), turned to 90 degrees
- moved C1 85.4 mm to (117.7, 82.3)
- moved TP1 84.0 mm to (113.5, 76.8)
- moved TP2 82.9 mm to (102.0, 89.0)
- moved R5 77.1 mm to (133.4, 79.2)
- moved C4 75.1 mm to (123.3, 79.3), turned to -90 degrees
- moved D1 72.4 mm to (133.4, 77.6)
- moved R4 68.8 mm to (121.8, 94.6), turned to 180 degrees
- moved U1 63.3 mm to (110.7, 76.8), turned to 90 degrees
- moved U2 57.8 mm to (117.5, 78.5), turned to 180 degrees
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Connections:
- C2 pad 1: +3.3V -> Net-(SW1-A)
- C4 pad 1: /Current Sensor/OUT -> +3.3V
- C6 pad 1: +3.3V -> Net-(U3--)
- C6 pad 2: GND -> /V_AMPLIFIED
- C7 pad 1: Net-(U4--) -> +3.3V
- C7 pad 2: /Amplifier/V_OUT -> GND
- C8 pad 1: Net-(SW3-A) -> /Current Sensor/OUT
- FB1 pad 1: Net-(U3-VOUT) -> Net-(U2-VOUT)
- R4 pad 2: Net-(U1-OUT) -> /OUT_FILT
- R6 pad 1: Net-(U4--) -> GND_VIRT
- R6 pad 2: /Amplifier/V_OUT -> Net-(U3--)
- R7 pad 1: GND_VIRT -> Net-(U3--)
- R7 pad 2: Net-(U4--) -> /V_AMPLIFIED
- R8 pad 2: /Amplifier/V_IN -> Net-(U4-OUT)
- SW1 pad 1: /Amplifier/V_OUT -> Net-(SW1-A)
- SW1 pad 2: Net-(J4-In) -> /OUT_FILT
- SW1 pad 3: /Amplifier/V_IN -> unconnected-(SW1-C-Pad3)
- TP2 pad 1: +3.3V -> GND
- U1 pad 1: /Current Sensor/IP+ -> +5V
- U1 pad 2: /Current Sensor/IP+ -> GND
- U1 pad 3: /Current Sensor/IP- -> +5V
- U1 pad 4: /Current Sensor/IP- -> +5V
- U1 pad 5: GND -> (no net)
- U1 pad 6: GND_VIRT -> +5V
- U2 pad 1: +5V -> GND
- U2 pad 2: GND -> +5V
- U2 pad 3: +5V -> Net-(U2-VOUT)
- U3 pad 1: GND -> /V_AMPLIFIED
- U3 pad 2: +5V -> GND
- U3 pad 3: Net-(U3-VOUT) -> /OUT_FILT
- U4 pad 1: /Amplifier/V_OUT -> /Current Sensor/IP+
- U4 pad 2: GND -> /Current Sensor/IP+
- U4 pad 3: /Amplifier/V_IN -> /Current Sensor/IP-
- U4 pad 4: Net-(U4--) -> /Current Sensor/IP-
- U4 pad 5: +3.3V -> GND
Routing:
- net +5V: track 0.00 -> 24.8 mm
- net GND: track 0.00 -> 18.1 mm, vias 0 -> 7
- net /OUT_FILT: track 0.00 -> 14.5 mm, vias 0 -> 1
- net /V_AMPLIFIED: track 0.00 -> 13.4 mm
- net /USB_SHIELD: track 0.00 -> 12.2 mm
- net +3.3V: track 0.00 -> 10.8 mm
- net Net-(J3-In): track 0.00 -> 10.7 mm, vias 0 -> 1
- net /Current Sensor/OUT: track 0.00 -> 9.99 mm
- net /CC1: track 0.00 -> 7.12 mm, vias 0 -> 2
- net /CC2: track 0.00 -> 7.09 mm, vias 0 -> 2
- net Net-(U3--): track 0.00 -> 4.71 mm
- net Net-(U4-OUT): track 0.00 -> 2.34 mm
- net Net-(SW1-A): track 0.00 -> 2.00 mm
- net Net-(U2-VOUT): track 0.00 -> 1.86 mm
- net Net-(D1-A): track 0.00 -> 1.61 mm
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- added copper zone on B.Cu, net GND
- added copper zone on F.Cu, net GND
- added copper zone on B.Cu, net GND_VIRT
- added copper zone on F.Cu, net GND_VIRT
Other:
- board outline added: 40 x 25 mm
- board text added: "+"
- board text added: "IN+"
- board text added: "IN-"
- board text added: "OFF"
- board text added: "ON"

Commit message: Rev A sent for manufacture.
Parts:
- moved U1 0.44 mm to (110.6, 77.2), turned to 0 degrees
- moved TP5 0.35 mm to (112.5, 94.0)
- moved TP6 0.35 mm to (106.5, 94.0)
- moved TP7 0.35 mm to (109.5, 94.0)
- moved C2 0.35 mm to (117.2, 94.2)
- moved R4 0.35 mm to (121.8, 94.2)
- moved SW1 0.35 mm to (120.2, 97.7)
- moved SW2 0.35 mm to (109.5, 97.7)
Routing:
- net +3.3V: track 10.8 -> 55.5 mm, vias 0 -> 1
- net GND_VIRT: track 0.00 -> 26.7 mm, vias 6 -> 12
- net /USB_SHIELD: track 12.2 -> 21.1 mm
- net /OUT_FILT: track 14.5 -> 19.6 mm
- net GND: track 18.1 -> 17.1 mm, vias 7 -> 53
- net +5V: track 24.8 -> 23.9 mm
- net /V_AMPLIFIED: track 13.4 -> 12.8 mm
- added copper zone on B.Cu, net /Current Sensor/IP+
- added copper zone on F.Cu, net /Current Sensor/IP+
- added copper zone on B.Cu, net /Current Sensor/IP-
- added copper zone on F.Cu, net /Current Sensor/IP-
